File: Electronic_Door_Lock.brd (EAGLE design)
At the start: 153.9 x 109.5 mm, 7 parts, among them U1 ARDUINO-UNO-R3-SHIELD

Commit message: Add files via upload
Parts:
- removed KEYPAD1: KEYPAD-4X4, Tinkercad:1X08
- added U2: IR-RECEIVERTSOP48, Tinkercad:TSOP48
Connections:
- removed net U1_D3: KEYPAD1.2, U1.D3
- removed net U1_D4: KEYPAD1.3, U1.D4
- removed net U1_D5: KEYPAD1.4, U1.D5
- removed net U1_D6: KEYPAD1.5, U1.D6
- removed net U1_D7: KEYPAD1.6, U1.D7
- removed net U1_D8: KEYPAD1.7, U1.D8
- removed net U1_D9: KEYPAD1.8, U1.D9
- net U1_5V: now also U2.3
- net U1_D2: now also U2.1; no longer KEYPAD1.1
- net U1_GND: now also U2.2
Changed lines of the file:
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@@
 </autorouter>
 <elements>
-<element name="SERVO1" library="Tinkercad" library_urn="urn:adsk.eagle:library:30890021" package="SG90" package3d_urn="urn:adsk.eagle:package:32659983/2" value="SERVOSG90" x="7.0612" y="62.6803" smashed="yes"/>
-<element name="KEYPAD1" library="Tinkercad" library_urn="urn:adsk.eagle:library:30890021" package="1X08" package3d_urn="urn:adsk.eagle:package:22409/2" value="KEYPAD-4X4" x="114.1271" y="71.6558" smashed="yes"/>
-<element name="U1" library="Tinkercad" library_urn="urn:adsk.eagle:library:30890021" package="ARDUINO-UNO-R3-SHIELD" package3d_urn="urn:adsk.eagle:package:32092383/4" value="ARDUINO-UNO-R3-SHIELD" x="119.3682" y="29.845" rot="R270" smashed="yes"/>
 <element name="R2" library="Tinkercad" library_urn="urn:adsk.eagle:library:30890021" package="RESAD1016W63L850D250B" package3d_urn="urn:adsk.eagle:package:31513020/2" value="220" x="44.1687" y="91.9787" rot="R90" smashed="yes"/>
 <element name="R1" library="Tinkercad" library_urn="urn:adsk.eagle:library:30890021" package="RESAD1016W63L850D250B" package3d_urn="urn:adsk.eagle:package:31513020/2" value="220" x="39.1873" y="92.212" rot="R90" smashed="yes"/>
 <element name="D1" library="Tinkercad" library_urn="urn:adsk.eagle:library:30890021" package="LED-RGB-5MM" package3d_urn="urn:adsk.eagle:package:32251353/4" value="LED-RGBRCBG-PTH" x="42.9688" y="101.9674" smashed="yes"/>
 <element name="R3" library="Tinkercad" library_urn="urn:adsk.eagle:library:30890021" package="RESAD1016W63L850D250B" package3d_urn="urn:adsk.eagle:package:31513020/2" value="220" x="46.9848" y="83.309" rot="R90" smashed="yes"/>
+<element name="U1" library="Tinkercad" library_urn="urn:adsk.eagle:library:30890021" package="ARDUINO-UNO-R3-SHIELD" package3d_urn="urn:adsk.eagle:package:32092383/4" value="ARDUINO-UNO-R3-SHIELD" x="119.3682" y="29.845" rot="R270" smashed="yes"/>
+<element name="U2" library="Tinkercad" library_urn="urn:adsk.eagle:library:30890021" package="TSOP48" package3d_urn="urn:adsk.eagle:package:32501402/2" value="IR-RECEIVERTSOP48" x="142.3644" y="64.3697" smashed="yes"/>
+<element name="SERVO1" library="Tinkercad" library_urn="urn:adsk.eagle:library:30890021" package="SG90" package3d_urn="urn:adsk.eagle:package:32659983/2" value="SERVOSG90" x="7.0612" y="62.6803" smashed="yes"/>
 </elements>
 <signals>
+<signal name="D1_B">
+<contactref element="D1" pad="B"/>
+<contactref element="R2" pad="2"/>
+<wire x1="43.6038" y1="102.6024" x2="44.1687" y2="97.0587" width="0" layer="19" extent="1-1"/>
+</signal>
+<signal name="U1_D13">
+<contactref element="R2" pad="1"/>
+<contactref element="U1" pad="D13"/>
+<wire x1="44.1687" y1="86.8987" x2="110.4782" y2="53.975" width="0" layer="19" extent="1-1"/>
+</signal>
+<signal name="D1_R">
+<contactref element="D1" pad="R"/>
+<contactref element="R1" pad="2"/>
+<wire x1="41.0638" y1="102.6024" x2="39.1873" y2="97.292" width="0" layer="19" extent="1-1"/>
+</signal>
+<signal name="U1_D11">
+<contactref element="R1" pad="1"/>
+<contactref element="U1" pad="D11"/>
+<wire x1="39.1873" y1="87.132" x2="115.5582" y2="53.975" width="0" layer="19" extent="1-1"/>
+</signal>
 <signal name="U1_GND">
 <contactref element="SERVO1" pad="1"/>
@@
 <contactref element="U1" pad="GND@2"/>
 <contactref element="D1" pad="C"/>
+<contactref element="U2" pad="2"/>
 <wire x1="121.9082" y1="5.715" x2="124.4482" y2="5.715" width="0" layer="19" extent="1-1"/>
 <wire x1="121.9082" y1="5.715" x2="107.9382" y2="53.975" width="0" layer="19" extent="1-1"/>
+<wire x1="107.9382" y1="53.975" x2="142.3644" y2="64.3697" width="0" layer="19" extent="1-1"/>
 <wire x1="107.9382" y1="53.975" x2="42.3338" y2="101.3324" width="0" layer="19" extent="1-1"/>
 <wire x1="4.5212" y1="62.6803" x2="42.3338" y2="101.3324" width="0" layer="19" extent="1-1"/>
+</signal>
+<signal name="D1_G">
+<contactref element="D1" pad="G"/>
+<contactref element="R3" pad="2"/>
+<wire x1="44.8738" y1="101.3324" x2="46.9848" y2="88.389" width="0" layer="19" extent="1-1"/>
+</signal>
+<signal name="U1_D12">
+<contactref element="R3" pad="1"/>
+<contactref element="U1" pad="D12"/>
+<wire x1="46.9848" y1="78.229" x2="113.0182" y2="53.975" width="0" layer="19" extent="1-1"/>
 </signal>
 <signal name="U1_D10">
@@
 <wire x1="9.6012" y1="62.6803" x2="118.0982" y2="53.975" width="0" layer="19" extent="1-1"/>
 </signal>
+<signal name="U1_D2">
+<contactref element="U2" pad="1"/>
+<contactref element="U1" pad="D2"/>
+<wire x1="139.8244" y1="64.3697" x2="139.6882" y2="53.975" width="0" layer="19" extent="1-1"/>
+</signal>
 <signal name="U1_5V">
 <contactref element="SERVO1" pad="2"/>
 <contactref element="U1" pad="5V"/>
+<contactref element="U2" pad="3"/>
+<wire x1="119.3682" y1="5.715" x2="144.9044" y2="64.3697" width="0" layer="19" extent="1-1"/>
 <wire x1="7.0612" y1="62.6803" x2="119.3682" y2="5.715" width="0" layer="19" extent="1-1"/>
 </signal>
-<signal name="U1_D6">
-<contactref element="KEYPAD1" pad="5"/>
-<contactref element="U1" pad="D6"/>
-<wire x1="115.3971" y1="71.6558" x2="129.5282" y2="53.975" width="0" layer="19" extent="1-1"/>
-</signal>
-<signal name="U1_D7">
-<contactref element="KEYPAD1" pad="6"/>
-<contactref element="U1" pad="D7"/>
-<wire x1="117.9371" y1="71.6558" x2="126.9882" y2="53.975" width="0" layer="19" extent="1-1"/>
-</signal>
-<signal name="U1_D8">
-<contactref element="KEYPAD1" pad="7"/>
-<contactref element="U1" pad="D8"/>
-<wire x1="120.4771" y1="71.6558" x2="123.1782" y2="53.975" width="0" layer="19" extent="1-1"/>
-</signal>
-<signal name="U1_D9">
-<contactref element="KEYPAD1" pad="8"/>
-<contactref element="U1" pad="D9"/>
-<wire x1="123.0171" y1="71.6558" x2="120.6382" y2="53.975" width="0" layer="19" extent="1-1"/>
-</signal>
-<signal name="U1_D5">
-<contactref element="KEYPAD1" pad="4"/>
-<contactref element="U1" pad="D5"/>
-<wire x1="112.8571" y1="71.6558" x2="132.0682" y2="53.975" width="0" layer="19" extent="1-1"/>
-</signal>
-<signal name="U1_D4">
-<contactref element="KEYPAD1" pad="3"/>
-<contactref element="U1" pad="D4"/>
-<wire x1="110.3171" y1="71.6558" x2="134.6082" y2="53.975" width="0" layer="19" extent="1-1"/>
-</signal>
-<signal name="U1_D3">
-<contactref element="KEYPAD1" pad="2"/>
-<contactref element="U1" pad="D3"/>
-<wire x1="107.7771" y1="71.6558" x2="137.1482" y2="53.975" width="0" layer="19" extent="1-1"/>
-</signal>
-<signal name="U1_D2">
-<contactref element="KEYPAD1" pad="1"/>
-<contactref element="U1" pad="D2"/>
-<wire x1="105.2371" y1="71.6558" x2="139.6882" y2="53.975" width="0" layer="19" extent="1-1"/>
-</signal>
-<signal name="U1_D13">
-<contactref element="R2" pad="1"/>
-<contactref element="U1" pad="D13"/>
-<wire x1="44.1687" y1="86.8987" x2="110.4782" y2="53.975" width="0" layer="19" extent="1-1"/>
-</signal>
-<signal name="U1_D12">
-<contactref element="R3" pad="1"/>
-<contactref element="U1" pad="D12"/>
-<wire x1="46.9848" y1="78.229" x2="113.0182" y2="53.975" width="0" layer="19" extent="1-1"/>
-</signal>
-<signal name="U1_D11">
-<contactref element="R1" pad="1"/>
-<contactref element="U1" pad="D11"/>
-<wire x1="39.1873" y1="87.132" x2="115.5582" y2="53.975" width="0" layer="19" extent="1-1"/>
-</signal>
-<signal name="D1_B">
-<contactref element="D1" pad="B"/>
-<contactref element="R2" pad="2"/>
-<wire x1="43.6038" y1="102.6024" x2="44.1687" y2="97.0587" width="0" layer="19" extent="1-1"/>
-</signal>
-<signal name="D1_R">
-<contactref element="D1" pad="R"/>
-<contactref element="R1" pad="2"/>
-<wire x1="41.0638" y1="102.6024" x2="39.1873" y2="97.292" width="0" layer="19" extent="1-1"/>
-</signal>
-<signal name="D1_G">
-<contactref element="D1" pad="G"/>
-<contactref element="R3" pad="2"/>
-<wire x1="44.8738" y1="101.3324" x2="46.9848" y2="88.389" width="0" layer="19" extent="1-1"/>
-</signal>
 </signals>
